File: pcb/mainboard/tmds_in.kicad_sch (KiCad schematic)
At the start: 37 parts, among them J4 HDMI_C_1.3, U15 ADV7611, Y3 24MHz

Commit message: PCB r1p3
Parts:
- added C179: 100nF/50V, Capacitor_SMD:C_0402_1005Metric, symbol Device:C
- added R23, R31: 10K/1%, Resistor_SMD:R_0402_1005Metric, symbol Device:R
- added U10: MT9700, Package_TO_SOT_SMD:SOT-23-5, symbol symbols:MT9700
Connections:
- net +5V: now also C179.1, U10.5 (VIN); no longer R47.1
- net GND: now also C179.2, R23.1, R31.1, U10.2 (GND)
- new net: R31.2, U10.3 (SET)
- new net: R47.1, U10.1 (VOUT)
- new net HPD_EN: R23.2, U10.4 (EN)
Other:
- moved on the sheet: R16, R47, R49
