File: pcb/mainboard/power_mon.kicad_sch (KiCad schematic)
At the start: 29 parts, among them U21 INA3221, U22 INA3221, U27 INA3221

Commit message: Sync local PCB changes
Parts:
- C163, C164, C168, C169: value 470nF/25V -> 1nF/25V
- C91: value 100nF/50V -> 1nF/50V
Changed lines of the file:
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@@
 			)
 		)
-		(property "Value" "470nF/25V"
-			(at 209.55 69.85 90)
+		(property "Value" "1nF/25V"
+			(at 210.82 69.85 90)
 			(effects
 				(font
@@
 			)
 		)
-		(property "Value" "470nF/25V"
-			(at 209.55 54.61 90)
+		(property "Value" "1nF/25V"
+			(at 210.82 54.61 90)
 			(effects
 				(font
@@
 			)
 		)
-		(property "Value" "470nF/25V"
-			(at 209.55 85.09 90)
+		(property "Value" "1nF/25V"
+			(at 210.82 85.09 90)
 			(effects
 				(font
@@
 			)
 		)
-		(property "Value" "100nF/50V"
-			(at 204.47 115.57 90)
+		(property "Value" "1nF/50V"
+			(at 205.74 115.57 90)
 			(effects
 				(font
@@
 			)
 		)
-		(property "Value" "470nF/25V"
-			(at 209.55 100.33 90)
+		(property "Value" "1nF/25V"
+			(at 210.82 100.33 90)
 			(effects
 				(font
