File: pcb/34p-adapter-a/adapter.kicad_pcb (KiCad board)
At the start: 2 copper layers, 45 x 41 mm, 6 parts, among them J3 FH12-50S-0.5SH, J5 FH12-34S-0.5SH

Commit message: Sync local PCB changes
Parts:
- J3: value FH12-50S-0.5SH -> FPC-05F-50PH20
- J5: value FH12-34S-0.5SH -> FH34SRJ-34S-0.5SH; footprint footprints:Xunpu_FPC-05F-34PH20_1x34-1MP_P0.50mm_Horizontal -> footprints:Hirose_FH34SRJ-34S-0.5SH_1x34-1MP_P0.50mm_Horizontal
- moved J5 1.55 mm to (155.1, 64.9)
Routing:
- net (no net): track 0.00 -> 0.72 mm, vias 0 -> 1
- net GND: track 28.9 -> 28.2 mm, vias 47 -> 46
Other:
- board text added: "Glider 34P-A Adapter Modos r0.3 251023"
- board text removed: "Glider 34P-A Adapter Modos r0.2 250428"
