File: pcb/34p-adapter-a/adapter.kicad_sch (KiCad schematic)
At the start: 8 parts, among them J3 FH12-50S-0.5SH, J5 FH12-34S-0.5SH

Commit message: Sync local PCB changes
Parts:
- J3: value FH12-50S-0.5SH -> FPC-05F-50PH20
- J5: value FH12-34S-0.5SH -> FH34SRJ-34S-0.5SH; footprint footprints:Xunpu_FPC-05F-34PH20_1x34-1MP_P0.50mm_Horizontal -> footprints:Hirose_FH34SRJ-34S-0.5SH_1x34-1MP_P0.50mm_Horizontal
Changed lines of the file:
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@@
 	(label "PGDSP"
 		(at 71.12 68.58 0)
-		(fields_autoplaced yes)
 		(effects
 			(font
@@
 	(label "SDCE0"
 		(at 177.8 71.12 0)
-		(fields_autoplaced yes)
 		(effects
 			(font
@@
 	(label "ED5"
 		(at 109.22 119.38 180)
-		(fields_autoplaced yes)
 		(effects
 			(font
@@
 	(label "ED1"
 		(at 177.8 76.2 0)
-		(fields_autoplaced yes)
 		(effects
 			(font
@@
 	(label "PD0"
 		(at 71.12 137.16 0)
-		(fields_autoplaced yes)
 		(effects
 			(font
@@
 	(label "SDCE0"
 		(at 109.22 63.5 180)
-		(fields_autoplaced yes)
 		(effects
 			(font
@@
 	(label "ESDLE"
 		(at 177.8 66.04 0)
-		(fields_autoplaced yes)
 		(effects
 			(font
@@
 	(label "PD6"
 		(at 71.12 114.3 0)
-		(fields_autoplaced yes)
 		(effects
 			(font
@@
 	(label "PSDCLK"
 		(at 71.12 76.2 0)
-		(fields_autoplaced yes)
 		(effects
 			(font
@@
 	(label "ED1"
 		(at 109.22 134.62 180)
-		(fields_autoplaced yes)
 		(effects
 			(font
@@
 	(label "PD9"
 		(at 71.12 104.14 0)
-		(fields_autoplaced yes)
 		(effects
 			(font
@@
 	(label "ED4"
 		(at 177.8 83.82 0)
-		(fields_autoplaced yes)
 		(effects
 			(font
@@
 	(label "ESDCLK"
 		(at 109.22 76.2 180)
-		(fields_autoplaced yes)
 		(effects
 			(font
@@
 	(label "PGDOE"
 		(at 71.12 66.04 0)
-		(fields_autoplaced yes)
 		(effects
 			(font
@@
 	(label "PD10"
 		(at 71.12 99.06 0)
-		(fields_autoplaced yes)
 		(effects
 			(font
@@
 	(label "PD5"
 		(at 71.12 119.38 0)
-		(fields_autoplaced yes)
 		(effects
 			(font
@@
 	(label "ESDCLK"
 		(at 177.8 60.96 0)
-		(fields_autoplaced yes)
 		(effects
 			(font
@@
 	(label "GDCLK"
 		(at 109.22 71.12 180)
-		(fields_autoplaced yes)
 		(effects
 			(font
@@
 	(label "ED9"
 		(at 109.22 104.14 180)
-		(fields_autoplaced yes)
 		(effects
 			(font
@@
 	(label "ESDOE"
 		(at 109.22 58.42 180)
-		(fields_autoplaced yes)
 		(effects
 			(font
@@
 	(label "ED12"
 		(at 109.22 91.44 180)
-		(fields_autoplaced yes)
 		(effects
 			(font
@@
 	(label "GDOE"
 		(at 109.22 66.04 180)
-		(fields_autoplaced yes)
 		(effects
 			(font
@@
 	(label "PD2"
 		(at 71.12 129.54 0)
-		(fields_autoplaced yes)
 		(effects
 			(font
@@
 	(label "ED13"
 		(at 109.22 88.9 180)
-		(fields_autoplaced yes)
 		(effects
 			(font
@@
 	(label "ESDOE"
 		(at 177.8 68.58 0)
-		(fields_autoplaced yes)
 		(effects
 			(font
@@
 	(label "PD11"
 		(at 71.12 96.52 0)
-		(fields_autoplaced yes)
 		(effects
 			(font
@@
 	(label "ED0"
 		(at 177.8 73.66 0)
-		(fields_autoplaced yes)
 		(effects
 			(font
@@
 	(label "ED14"
 		(at 109.22 86.36 180)
-		(fields_autoplaced yes)
 		(effects
 			(font
@@
 	(label "ED6"
 		(at 109.22 116.84 180)
-		(fields_autoplaced yes)
 		(effects
 			(font
@@
 	(label "ED7"
 		(at 177.8 91.44 0)
-		(fields_autoplaced yes)
 		(effects
 			(font
@@
 	(label "ED0"
 		(at 109.22 137.16 180)
-		(fields_autoplaced yes)
 		(effects
 			(font
@@
 	(label "ED4"
 		(at 109.22 121.92 180)
-		(fields_autoplaced yes)
 		(effects
 			(font
@@
 	(label "GDOE"
 		(at 177.8 109.22 0)
-		(fields_autoplaced yes)
 		(effects
 			(font
@@
 	(label "PD1"
 		(at 71.12 134.62 0)
-		(fields_autoplaced yes)
 		(effects
 			(font
@@
 	(label "PSDCE0"
 		(at 71.12 63.5 0)
-		(fields_autoplaced yes)
 		(effects
 			(font
@@
 	(label "ED11"
 		(at 109.22 99.06 180)
-		(fields_autoplaced yes)
 		(effects
 			(font
@@
 	(label "PD15"
 		(at 71.12 81.28 0)
-		(fields_autoplaced yes)
 		(effects
 			(font
@@
 	(label "ED10"
 		(at 109.22 101.6 180)
-		(fields_autoplaced yes)
 		(effects
 			(font
@@
 	(label "PSDOE"
 		(at 71.12 58.42 0)
-		(fields_autoplaced yes)
 		(effects
 			(font
@@
 	(label "PD7"
 		(at 71.12 111.76 0)
-		(fields_autoplaced yes)
 		(effects
 			(font
@@
 	(label "ED2"
 		(at 177.8 78.74 0)
-		(fields_autoplaced yes)
 		(effects
 			(font
@@
 	(label "ED7"
 		(at 109.22 114.3 180)
-		(fields_autoplaced yes)
 		(effects
 			(font
@@
 	(label "BORDER"
 		(at 175.26 119.38 0)
-		(fields_autoplaced yes)
 		(effects
 			(font
@@
 	(label "ED2"
 		(at 109.22 132.08 180)
-		(fields_autoplaced yes)
 		(effects
 			(font
@@
 	(label "GDCLK"
 		(at 177.8 111.76 0)
-		(fields_autoplaced yes)
 		(effects
 			(font
@@
 	(label "GDSP"
 		(at 177.8 114.3 0)
-		(fields_autoplaced yes)
 		(effects
 			(font
@@
 	(label "ED6"
 		(at 177.8 88.9 0)
-		(fields_autoplaced yes)
 		(effects
 			(font
@@
 	(label "ED8"
 		(at 109.22 106.68 180)
-		(fields_autoplaced yes)
 		(effects
 			(font
@@
 	(label "ED3"
 		(at 109.22 129.54 180)
-		(fields_autoplaced yes)
 		(effects
 			(font
@@
 	(label "PD3"
 		(at 71.12 127 0)
-		(fields_autoplaced yes)
 		(effects
 			(font
@@
 	(label "ESDLE"
 		(at 109.22 60.96 180)
-		(fields_autoplaced yes)
 		(effects
 			(font
@@
 	(label "PD13"
 		(at 71.12 88.9 0)
-		(fields_autoplaced yes)
 		(effects
 			(font
@@
 	(label "PD8"
 		(at 71.12 106.68 0)
-		(fields_autoplaced yes)
 		(effects
 			(font
@@
 	(label "ED3"
 		(at 177.8 81.28 0)
-		(fields_autoplaced yes)
 		(effects
 			(font
@@
 	(label "BORDER"
 		(at 236.22 152.4 0)
-		(fields_autoplaced yes)
 		(effects
 			(font
@@
 	(label "ED15"
 		(at 109.22 83.82 180)
-		(fields_autoplaced yes)
 		(effects
 			(font
@@
 	(label "PD12"
 		(at 71.12 91.44 0)
-		(fields_autoplaced yes)
 		(effects
 			(font
@@
 	(label "PD14"
 		(at 71.12 83.82 0)
-		(fields_autoplaced yes)
 		(effects
 			(font
@@
 	(label "GDSP"
 		(at 109.22 68.58 180)
-		(fields_autoplaced yes)
 		(effects
 			(font
@@
 	(label "ED5"
 		(at 177.8 86.36 0)
-		(fields_autoplaced yes)
 		(effects
 			(font
@@
 	(label "PSDLE"
 		(at 71.12 60.96 0)
-		(fields_autoplaced yes)
 		(effects
 			(font
@@
 	(label "PD4"
 		(at 71.12 121.92 0)
-		(fields_autoplaced yes)
 		(effects
 			(font
@@
 	(label "PGDCLK"
 		(at 71.12 71.12 0)
-		(fields_autoplaced yes)
 		(effects
 			(font
@@
 			)
 		)
-		(property "Value" "FH12-34S-0.5SH"
+		(property "Value" "FH34SRJ-34S-0.5SH"
 			(at 180.34 39.37 0)
 			(effects
@@
 			)
 		)
-		(property "Footprint" "footprints:Xunpu_FPC-05F-34PH20_1x34-1MP_P0.50mm_Horizontal"
+		(property "Footprint" "footprints:Hirose_FH34SRJ-34S-0.5SH_1x34-1MP_P0.50mm_Horizontal"
 			(at 193.04 83.82 0)
 			(effects
@@
 			)
 		)
-		(property "Value" "FH12-50S-0.5SH"
+		(property "Value" "FPC-05F-50PH20"
 			(at 74.93 36.83 0)
 			(effects
