File: pcb/mega_adapter/adapter.kicad_pcb (KiCad board)
At the start: 2 copper layers, 59 x 44 mm, 18 parts, among them J1 AFC24-S40FIA-00, J11 32P Lower Contact, J3 FH12-50S-0.5SH, J4 FH12-33S-0.5SH, J5 FH12-34S-0.5SH, J6 502598-3993, J9 FH28-50S-0.5SH

Commit message: PCB r1p3
Parts:
- removed J11: 32P Lower Contact, footprints:Hirose_FH12-32S-0.5SH_1x32-1MP_P0.50mm_Horizontal_Mirrored
- removed R8: 0, Resistor_SMD:R_0402_1005Metric
Routing:
- net GND: track 230.4 -> 183.8 mm, vias 38 -> 34
- net -VCOM: track 158.4 -> 134.5 mm, vias 12 -> 11
- net /PSDLE: track 24.6 -> 2.25 mm, vias 2 -> 0
- net /PSDCE0: track 24.5 -> 2.25 mm, vias 2 -> 0
- net /PSDOE: track 24.3 -> 2.25 mm, vias 2 -> 0
- net -VGL: track 134.1 -> 112.8 mm
- net +3V3: track 179.4 -> 159.3 mm
- net /PSDCLK: track 21.5 -> 2.32 mm, vias 2 -> 0
- net +VGH: track 147.8 -> 129.1 mm
- net +VP: track 129.7 -> 114.7 mm, vias 7 -> 6
- net -VN: track 139.1 -> 125.4 mm, vias 5 -> 4
- net /PGDOE: track 14.3 -> 2.25 mm
- net /PD1: track 13.8 -> 2.40 mm
- net /PD0: track 13.8 -> 2.40 mm
- net /PD3: track 13.4 -> 2.19 mm
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Other:
- board size 59 x 44 mm -> 59 x 40.9 mm

Commit message: Sync local PCB changes
Parts:
- J3: footprint footprints:Hirose_FH12-50S-0.5SH_1x50-1MP_P0.50mm_Horizontal_Mirrored -> footprints:Xunpu_FPC-05F-50PH20_1x50-1MP_P0.50mm_Horizontal_Mirrored
- J4: value FH12-33S-0.5SH -> FPC-05F-33PH20; footprint Connector_FFC-FPC:Hirose_FH12-33S-0.5SH_1x33-1MP_P0.50mm_Horizontal -> footprints:Xunpu_FPC-05F-33PH20_1x33-1MP_P0.50mm_Horizontal
- J5: value FH12-34S-0.5SH -> FH34SRJ-34S-0.5SH; footprint Connector_FFC-FPC:Hirose_FH12-34S-0.5SH_1x34-1MP_P0.50mm_Horizontal -> footprints:Hirose_FH34SRJ-34S-0.5SH_1x34-1MP_P0.50mm_Horizontal
- J9: footprint Connector_FFC-FPC:Hirose_FH12-50S-0.5SH_1x50-1MP_P0.50mm_Horizontal -> footprints:Xunpu_FPC-05F-50PH20_1x50-1MP_P0.50mm_Horizontal
- moved J5 0.55 mm to (188.2, 57.5)
Routing:
- net GND: track 183.8 -> 196.8 mm, vias 34 -> 35
- net -VCOM: track 134.5 -> 140.1 mm
- net /ED1: track 131.1 -> 133.9 mm
- net /ED5: track 122.0 -> 124.8 mm
- net /ED4: track 122.0 -> 124.9 mm
- net /ED3: track 123.9 -> 126.7 mm
- net /ED2: track 125.5 -> 128.3 mm
- net /ED0: track 131.1 -> 133.9 mm
- net +VP: track 114.7 -> 117.6 mm
- net +VGH: track 129.1 -> 131.9 mm
- net /ED7: track 121.2 -> 124.0 mm
- net /SDCE0: track 156.4 -> 153.7 mm
- net /GDCLK: track 142.2 -> 139.5 mm
- net /ESDOE: track 162.4 -> 159.6 mm
- net /ESDCLK: track 145.9 -> 143.1 mm
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Other:
- board text added: "Contact facing down!"
