File: pcb/mega_adapter/adapter.kicad_sch (KiCad schematic)
At the start: 18 parts, among them J1 AFC24-S40FIA-00, J11 32P Lower Contact, J3 FH12-50S-0.5SH, J4 FH12-33S-0.5SH, J5 FH12-34S-0.5SH, J6 502598-3993, J9 FH28-50S-0.5SH

Commit message: PCB r1p3
Parts:
- removed J11: 32P Lower Contact, footprints:Hirose_FH12-32S-0.5SH_1x32-1MP_P0.50mm_Horizontal_Mirrored, symbol Connector_Generic_MountingPin:Conn_01x32_MountingPin
- removed R8: 0, Resistor_SMD:R_0402_1005Metric, symbol Device:R

Commit message: Sync local PCB changes
Parts:
- J3: footprint footprints:Hirose_FH12-50S-0.5SH_1x50-1MP_P0.50mm_Horizontal_Mirrored -> footprints:Xunpu_FPC-05F-50PH20_1x50-1MP_P0.50mm_Horizontal_Mirrored
- J4: value FH12-33S-0.5SH -> FPC-05F-33PH20; footprint Connector_FFC-FPC:Hirose_FH12-33S-0.5SH_1x33-1MP_P0.50mm_Horizontal -> footprints:Xunpu_FPC-05F-33PH20_1x33-1MP_P0.50mm_Horizontal
- J5: value FH12-34S-0.5SH -> FH34SRJ-34S-0.5SH; footprint Connector_FFC-FPC:Hirose_FH12-34S-0.5SH_1x34-1MP_P0.50mm_Horizontal -> footprints:Hirose_FH34SRJ-34S-0.5SH_1x34-1MP_P0.50mm_Horizontal
- J9: footprint Connector_FFC-FPC:Hirose_FH12-50S-0.5SH_1x50-1MP_P0.50mm_Horizontal -> footprints:Xunpu_FPC-05F-50PH20_1x50-1MP_P0.50mm_Horizontal
Changed lines of the file:
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@@
 			)
 		)
-		(property "Footprint" "Connector_FFC-FPC:Hirose_FH12-50S-0.5SH_1x50-1MP_P0.50mm_Horizontal"
+		(property "Footprint" "footprints:Xunpu_FPC-05F-50PH20_1x50-1MP_P0.50mm_Horizontal"
 			(at 342.9 99.06 0)
 			(effects
@@
 			)
 		)
-		(property "Value" "FH12-34S-0.5SH"
+		(property "Value" "FH34SRJ-34S-0.5SH"
 			(at 187.96 34.29 0)
 			(effects
@@
 			)
 		)
-		(property "Footprint" "Connector_FFC-FPC:Hirose_FH12-34S-0.5SH_1x34-1MP_P0.50mm_Horizontal"
+		(property "Footprint" "footprints:Hirose_FH34SRJ-34S-0.5SH_1x34-1MP_P0.50mm_Horizontal"
 			(at 200.66 78.74 0)
 			(effects
@@
 			)
 		)
-		(property "Value" "FH12-33S-0.5SH"
+		(property "Value" "FPC-05F-33PH20"
 			(at 222.25 34.29 0)
 			(effects
@@
 			)
 		)
-		(property "Footprint" "Connector_FFC-FPC:Hirose_FH12-33S-0.5SH_1x33-1MP_P0.50mm_Horizontal"
+		(property "Footprint" "footprints:Xunpu_FPC-05F-33PH20_1x33-1MP_P0.50mm_Horizontal"
 			(at 236.22 78.74 0)
 			(effects
@@
 			)
 		)
-		(property "Footprint" "footprints:Hirose_FH12-50S-0.5SH_1x50-1MP_P0.50mm_Horizontal_Mirrored"
+		(property "Footprint" "footprints:Xunpu_FPC-05F-50PH20_1x50-1MP_P0.50mm_Horizontal_Mirrored"
 			(at 71.12 149.86 0)
 			(effects
